File: GETWAY_v2.kicad_pcb (KiCad board)
At the start: 2 copper layers, 100 x 75 mm, 232 parts, among them IC2 MP1584EN, J1 STM_MicroSD_Socket, J10 SWD, J11 ANT2, J12 ESP_MicroSD_Socket, J14 ESP_ANTENA, J15 LORA_ANTENA, J16 ANT1, J3 FPC_32p, J4 HR911105A, J5 USB_C_UART, J6 USB_C_OTG, J7 CONNECTOR, J8 BAT, J9 AudioJack, Q1 BC847, Q2 BC847, SW1 STMRESET, SW2 ESP RESET, SW3 ESP BOOT, U1 STM32F407VGTx, U10 USBLC6-2SC6, U11 CP2102N, U12 USBLC6-2SC6, U13 LTV-817S, U14 LTV-817S, U15 LM358, U16 AMS1117-3.3, U2 ESP32-WROOM-32U, U3 Ai-Thinker-Ra-02, U4 W25Q32JVSS, U5 74HC04, U6 MAX485E, U7 DS3231M, U8 LAN8720A, U9 UDA1334ATS, Y1 25MHz, Y2 25MHz

Commit message: Add files via upload
Parts:
- added C25: 10uF, Capacitor_SMD:C_1206_3216Metric, F.Cu at (142.4, 88.8)
- added J2: SPI, Connector_PinHeader_2.54mm:PinHeader_2x04_P2.54mm_Vertical, F.Cu at (134.1, 116.5)
- moved C30 9.33 mm to (130.4, 81.5)
- moved JP5 5.66 mm to (124.8, 84.8), turned to 180 degrees
- moved SW3 3.22 mm to (178.2, 122.0)
- moved JP4 1.76 mm to (149.6, 85.9)
- moved JP2 1.76 mm to (154.7, 85.9)
- moved JP3 1.76 mm to (152.2, 85.9)
- moved C1 1.50 mm to (91.3, 128.3)
- moved R3 1.50 mm to (91.3, 126.8)
- moved C7 1.05 mm to (169.4, 121.3)
- moved R6 1.05 mm to (169.4, 122.8)
- moved C48 0.13 mm to (142.4, 90.8)
Routing:
- net +3.3V: track 285.8 -> 493.7 mm, vias 13 -> 20
- net +5V: track 130.6 -> 270.1 mm, vias 7 -> 18
- net ESP_RESET: track 4.66 -> 85.4 mm, vias 0 -> 4
- net GND: track 276.6 -> 355.7 mm, vias 24 -> 47
- net USART1_TX: track 29.9 -> 87.1 mm, vias 5 -> 3
- net BOOT-ETH_REFCLKO: track 50.5 -> 106.6 mm
- net USART1_RX: track 49.5 -> 103.4 mm, vias 7 -> 5
- net SPI1_CS1: track 3.58 -> 44.7 mm
- net SPI1_CS2: track 4.30 -> 44.9 mm
- net STM_I2S_CK: track 0.00 -> 29.3 mm, vias 0 -> 1
- net ESP_I2S_SD: track 9.33 -> 37.0 mm
- net RXD0: track 58.2 -> 85.7 mm, vias 2 -> 4
- net ESP_I2S_CK: track 10.0 -> 37.0 mm
- net Earth: track 8.82 -> 35.3 mm, vias 0 -> 1
- net STM_I2S_WS: track 0.00 -> 25.5 mm, vias 0 -> 1
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- added copper zone on F.Cu, net +3.3V
- added copper zone on F.Cu, net +5V
- added copper zone on F.Cu, net VCC
- removed copper zone on B.Cu, net Net-(C18-Pad1)
- removed copper zone on B.Cu, net Net-(C19-Pad1)

Commit message: Add files via upload
Parts:
- added C72: 100nF, Capacitor_SMD:C_0603_1608Metric, F.Cu at (106.8, 113.5)
- added C75: 10uF, Capacitor_SMD:C_1206_3216Metric, F.Cu at (131.9, 84.2)
- added C76: 10uF, Capacitor_SMD:C_1206_3216Metric, F.Cu at (116.4, 84.9)
- added C77: 10uF, Capacitor_SMD:C_1206_3216Metric, F.Cu at (112.5, 73.9)
- added C78: 47uF, Capacitor_SMD:CP_Elec_5x5.4, F.Cu at (162.5, 88.0)
- added C79: 47uF, Capacitor_SMD:CP_Elec_5x5.4, F.Cu at (156.7, 88.0)
- moved C62 3.03 mm to (168.6, 93.9), turned to 0 degrees
- moved C10 0.15 mm to (167.9, 95.9)
Routing:
- net GND: track 355.7 -> 436.6 mm, vias 47 -> 63
- net +5V: track 270.1 -> 340.0 mm, vias 18 -> 20
- net +3.3V: track 493.7 -> 539.7 mm, vias 20 -> 22
- net RS485_A: track 21.2 -> 30.2 mm
- net INPUT-: track 25.9 -> 31.6 mm
- net RXD0: track 85.7 -> 91.0 mm
- net TXD0: track 82.1 -> 86.7 mm
- net Net-(C62-Pad2): track 15.4 -> 11.6 mm
- net BOOT-ETH_REFCLKO: track 106.6 -> 110.3 mm
- net ESP_RESET: track 85.4 -> 87.1 mm
- net VCC: track 53.7 -> 52.8 mm
- net Net-(R23-Pad1): track 5.96 -> 5.13 mm
- net SWCLK: track 29.4 -> 28.7 mm
- net Net-(JP2-Pad2): track 7.19 -> 6.55 mm
- net SWDIO: track 29.7 -> 29.1 mm
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- added copper zone on F.Cu, net Net-(D6-Pad1)

Commit message: Add files via upload
Parts:
- added C80: 10uF, Capacitor_SMD:C_1206_3216Metric, F.Cu at (184.6, 98.1)
- added C81: 10uF, Capacitor_SMD:C_1206_3216Metric, F.Cu at (178.6, 98.1)
- moved C7 0.58 mm to (169.4, 120.7)
- moved R6 0.58 mm to (169.4, 122.2)
- turned J16 to -90 degrees
Routing:
- net GND: track 436.6 -> 423.6 mm, vias 63 -> 372
- net +3.3V: track 539.7 -> 543.0 mm
- net ESP_RESET: track 87.1 -> 87.9 mm
- net BOOT-ETH_REFCLKO: track 110.3 -> 109.7 mm
- net Net-(C21-Pad1): vias 1 -> 2
Other:
- board text added: "3V3"
- board text added: "BAT+"
- board text added: "BAT-"
- board text added: "CS1"
- board text added: "CS2"
- board text added: "Design by Mai Văn Anh"
- board text added: "EBOOT"
- board text added: "ERST"
- board text added: "MISO"
- board text added: "MOSI"
- board text added: "PC13"
- board text added: "SCK"
- board text added: "SPI1"
- board text added: "SRST"
- board text added: "SWCLK"
- board text added: "SWD"
- board text added: "SWDIO"
- board text removed: "BOOT0"
- board text removed: "By Mai Van Anh"
- board text removed: "ESP SD"
