File: POWER.kicad_sch (KiCad schematic)
At the start: 54 parts, among them IC2 MP1584EN, U16 AMS1117-3.3

Commit message: Add files via upload
Parts:
- added C25: 10uF, Capacitor_SMD:C_1206_3216Metric, symbol Device:C_Small
Connections:
- net +3.3V: now also C25.2
- net GND: now also C25.1
Changed lines of the file:
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@@
   (junction (at 118.11 99.695) (diameter 0) (color 0 0 0 0)
   )
+  (junction (at 245.11 99.695) (diameter 0) (color 0 0 0 0)
+  )
   (junction (at 72.39 111.125) (diameter 0) (color 0 0 0 0)
   )
@@
   (junction (at 224.79 99.695) (diameter 0) (color 0 0 0 0)
   )
+  (junction (at 245.11 111.125) (diameter 0) (color 0 0 0 0)
+  )
   (junction (at 123.19 99.695) (diameter 0) (color 0 0 0 0)
   )
@@
     (stroke (width 0) (type default) (color 0 0 0 0))
   )
+  (wire (pts (xy 250.19 104.775) (xy 250.19 99.695))
+    (stroke (width 0) (type default) (color 0 0 0 0))
+  )
+  (wire (pts (xy 250.19 99.695) (xy 245.11 99.695))
+    (stroke (width 0) (type default) (color 0 0 0 0))
+  )
   (wire (pts (xy 118.11 99.695) (xy 123.19 99.695))
     (stroke (width 0) (type default) (color 0 0 0 0))
@@
     (stroke (width 0) (type default) (color 0 0 0 0))
   )
+  (wire (pts (xy 250.19 109.855) (xy 250.19 111.125))
+    (stroke (width 0) (type default) (color 0 0 0 0))
+  )
   (wire (pts (xy 97.79 99.695) (xy 102.87 99.695))
     (stroke (width 0) (type default) (color 0 0 0 0))
@@
   )
   (wire (pts (xy 173.99 109.855) (xy 173.99 111.125))
+    (stroke (width 0) (type default) (color 0 0 0 0))
+  )
+  (wire (pts (xy 250.19 111.125) (xy 245.11 111.125))
     (stroke (width 0) (type default) (color 0 0 0 0))
   )
@@
       (effects (font (size 1.27 1.27)) hide)
     )
+    (pin "1")
+    (pin "2")
+  )
+  (symbol (lib_id "Device:C_Small") (at 250.19 107.315 0) (mirror x) (unit 1)
+    (in_bom yes) (on_board yes)
+    (property "Reference" "C25" (id 0) (at 252.73 108.585 90))
+    (property "Value" "10uF" (id 1) (at 252.73 103.505 90))
+    (property "Footprint" "Capacitor_SMD:C_1206_3216Metric" (id 2) (at 250.19 107.315 0)
+      (effects (font (size 1.27 1.27)) hide)
+    )
+    (property "Datasheet" "~" (id 3) (at 250.19 107.315 0)
+      (effects (font (size 1.27 1.27)) hide)
+    )

Commit message: Add files via upload
Parts:
- added C72: 100nF, Capacitor_SMD:C_0603_1608Metric, symbol Device:C_Small
- added C75, C76, C77: 10uF, Capacitor_SMD:C_1206_3216Metric, symbol Device:C_Small
- added C78, C79: 47uF, Capacitor_SMD:CP_Elec_5x5.4, symbol Device:C_Polarized_Small
Connections:
- net +3.3V: now also C76.2, C77.2, C79.1
- net +5V: now also C72.2, C75.2, C78.1
- net GND: now also C72.1, C75.1, C76.1, C77.1, C78.2, C79.2
Other:
- moved on the sheet: C23, C24, C25, C41, C71

Commit message: Add files via upload
Parts:
- added C80, C81: 10uF, Capacitor_SMD:C_1206_3216Metric, symbol Device:C_Small
Connections:
- net +3.3V: now also C80.2, C81.2
- net GND: now also C80.1, C81.1
Changed lines of the file:
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@@
   (junction (at 153.67 111.125) (diameter 0) (color 0 0 0 0)
   )
+  (junction (at 186.69 132.715) (diameter 0) (color 0 0 0 0)
+  )
   (junction (at 134.62 50.8) (diameter 0) (color 0 0 0 0)
   )
@@
   (junction (at 224.79 111.125) (diameter 0) (color 0 0 0 0)
   )
+  (junction (at 186.69 144.145) (diameter 0) (color 0 0 0 0)
+  )
   (junction (at 138.43 111.125) (diameter 0) (color 0 0 0 0)
   )
@@
   (junction (at 214.63 111.125) (diameter 0) (color 0 0 0 0)
   )
+  (junction (at 181.61 132.715) (diameter 0) (color 0 0 0 0)
+  )
   (junction (at 168.91 99.695) (diameter 0) (color 0 0 0 0)
   )
@@
   (junction (at 125.73 99.695) (diameter 0) (color 0 0 0 0)
   )
+  (junction (at 181.61 144.145) (diameter 0) (color 0 0 0 0)
+  )
   (junction (at 97.79 130.175) (diameter 0) (color 0 0 0 0)
   )
@@
     (stroke (width 0) (type default) (color 0 0 0 0))
   )
+  (wire (pts (xy 191.77 142.875) (xy 191.77 144.145))
+    (stroke (width 0) (type default) (color 0 0 0 0))
+  )
   (wire (pts (xy 204.47 111.125) (xy 209.55 111.125))
     (stroke (width 0) (type default) (color 0 0 0 0))
@@
     (stroke (width 0) (type default) (color 0 0 0 0))
   )
+  (wire (pts (xy 186.69 142.875) (xy 186.69 144.145))
+    (stroke (width 0) (type default) (color 0 0 0 0))
+  )
   (wire (pts (xy 204.47 99.695) (xy 204.47 104.775))
     (stroke (width 0) (type default) (color 0 0 0 0))
@@
     (stroke (width 0) (type default) (color 0 0 0 0))
   )
+  (wire (pts (xy 186.69 144.145) (xy 181.61 144.145))
+    (stroke (width 0) (type default) (color 0 0 0 0))
+  )
   (wire (pts (xy 179.07 99.695) (xy 184.15 99.695))
     (stroke (width 0) (type default) (color 0 0 0 0))
@@
     (stroke (width 0) (type default) (color 0 0 0 0))
   )
+  (wire (pts (xy 186.69 137.795) (xy 186.69 132.715))
+    (stroke (width 0) (type default) (color 0 0 0 0))
+  )
   (wire (pts (xy 181.61 132.715) (xy 176.53 132.715))
     (stroke (width 0) (type default) (color 0 0 0 0))
@@
     (stroke (width 0) (type default) (color 0 0 0 0))
   )
+  (wire (pts (xy 191.77 144.145) (xy 186.69 144.145))
+    (stroke (width 0) (type default) (color 0 0 0 0))
+  )
   (wire (pts (xy 60.325 99.695) (xy 60.325 104.775))
     (stroke (width 0) (type default) (color 0 0 0 0))
@@
     (stroke (width 0) (type default) (color 0 0 0 0))
   )
+  (wire (pts (xy 191.77 132.715) (xy 186.69 132.715))
+    (stroke (width 0) (type default) (color 0 0 0 0))
+  )
   (wire (pts (xy 118.11 111.125) (xy 123.19 111.125))
     (stroke (width 0) (type default) (color 0 0 0 0))
@@
     (stroke (width 0) (type default) (color 0 0 0 0))
   )
+  (wire (pts (xy 191.77 137.795) (xy 191.77 132.715))
+    (stroke (width 0) (type default) (color 0 0 0 0))
+  )
   (wire (pts (xy 97.79 99.695) (xy 97.79 104.775))
     (stroke (width 0) (type default) (color 0 0 0 0))
@@
   )
   (wire (pts (xy 173.99 99.695) (xy 179.07 99.695))
+    (stroke (width 0) (type default) (color 0 0 0 0))
+  )
+  (wire (pts (xy 186.69 132.715) (xy 181.61 132.715))
     (stroke (width 0) (type default) (color 0 0 0 0))
   )
@@
     )
     (property "Datasheet" "~" (id 3) (at 199.39 107.315 0)
+      (effects (font (size 1.27 1.27)) hide)
+    )
+    (pin "1")
+    (pin "2")
+  )
+  (symbol (lib_id "Device:C_Small") (at 186.69 140.335 0) (mirror x) (unit 1)
+    (in_bom yes) (on_board yes)
+    (property "Reference" "C80" (id 0) (at 189.23 141.605 90))
+    (property "Value" "10uF" (id 1) (at 189.23 136.525 90))
+    (property "Footprint" "Capacitor_SMD:C_1206_3216Metric" (id 2) (at 186.69 140.335 0)
+      (effects (font (size 1.27 1.27)) hide)
+    )
+    (property "Datasheet" "~" (id 3) (at 186.69 140.335 0)
       (effects (font (size 1.27 1.27)) hide)
     )
@@
       (effects (font (size 1.27 1.27)) hide)
     )
+    (pin "1")
+    (pin "2")
+  )
+  (symbol (lib_id "Device:C_Small") (at 191.77 140.335 0) (mirror x) (unit 1)
+    (in_bom yes) (on_board yes)
+    (property "Reference" "C81" (id 0) (at 194.31 141.605 90))
+    (property "Value" "10uF" (id 1) (at 194.31 136.525 90))
+    (property "Footprint" "Capacitor_SMD:C_1206_3216Metric" (id 2) (at 191.77 140.335 0)
+      (effects (font (size 1.27 1.27)) hide)
+    )
+    (property "Datasheet" "~" (id 3) (at 191.77 140.335 0)
+      (effects (font (size 1.27 1.27)) hide)
+    )
